Commit message: Changed Task Spline to Body Frame
Added appropriate change of transforms to be in body frame as opposed to world frame.

File: dogebot.urdf (robot description, URDF)
Before this commit: robot dogebot, 26 links, 25 joints
Links:
- removed link world
Joints:
- removed joint world_to_body
